Commit message: simulating front wheels in roboteq

File: komodo2_description/urdf/komodo2_gazebo.xacro (robot description, xacro)
@@ -96,5 +96,5 @@
                 <maxVel>1.0</maxVel>
                 <minDepth>0.00</minDepth>
-                <material>Gazebo/Black</material>
+<!--                <material>Gazebo/Black</material>-->
             </gazebo>
             <gazebo reference="front_right_wheel_link">
@@ -107,5 +107,5 @@
                 <maxVel>1.0</maxVel>
                 <minDepth>0.00</minDepth>
-                <material>Gazebo/Black</material>
+<!--                <material>Gazebo/Black</material>-->
             </gazebo>
             <gazebo reference="rear_left_wheel_link">
@@ -118,5 +118,5 @@
                 <maxVel>1.0</maxVel>
                 <minDepth>0.00</minDepth>
-                <material>Gazebo/Black</material>
+<!--                <material>Gazebo/Black</material>-->
             </gazebo>
             <gazebo reference="rear_right_wheel_link">
@@ -129,5 +129,5 @@
                 <maxVel>1.0</maxVel>
                 <minDepth>0.00</minDepth>
-                <material>Gazebo/Black</material>
+<!--                <material>Gazebo/Black</material>-->
             </gazebo>
             <gazebo reference="base_link">

Commit message: added depth cam to simulation

File: komodo2_description/urdf/komodo2_gazebo.xacro (robot description, xacro)
@@ -11,12 +11,12 @@
     <xacro:arg name="rgb_cam" default="false"/>
     <xacro:arg name="depth_cam" default="false"/>
-    <!-- softkinetic -->
-    <xacro:if value="$(arg rgb_cam)">
-<!--        <xacro:softkinetic_gazebo name="softkinetic_camera_rgb" ros_topic="softkinetic_camera"/> -->
-    </xacro:if>
     <!-- cameras  -->
     <xacro:if value="$(arg rgb_cam)">
         <xacro:Camera name="rgb_cam" link="rgb_cam_link" image_width="640" image_height="480"
                       image_format="R8G8B8" clip_near="0.02" clip_far="300" />
+        </xacro:if>
+        <xacro:if value="$(arg depth_cam)">
+           <xacro:include filename="$(find komodo2_gazebo)/macros/depth_cam.xacro" />
+            <xacro:softkinetic_gazebo name="softkinetic_rgb" ros_topic="softkinetic"/>
         </xacro:if>
         <!-- Sonars -->

File: komodo2_gazebo/macros/depth_cam.xacro (robot description, xacro)
@@ -1,50 +1,48 @@
 <?xml version="1.0"?>
 <robot xmlns:xacro="http://www.ros.org/wiki/xacro">
-  <xacro:macro name="depth_cam" params="name ros_topic">
-    <gazebo reference="${name}_frame">
-      <sensor type="depth" name="${name}_frame_sensor">
-        <always_on>true</always_on>
-        <update_rate>25.0</update_rate>
+  <xacro:macro name="softkinetic_gazebo" params="name ros_topic">
+ <!-- camera -->
+  <gazebo reference="camera_link">
+    <sensor type="depth" name="camera1">
+        <always_on>1</always_on>
+        <visualize>true</visualize>
         <camera>
-          <horizontal_fov>${74.0*M_PI/180.0}</horizontal_fov>
-          <image>
-            <format>B8G8R8</format>
-            <width>320</width>
-            <height>240</height>
-          </image>
-          <clip>
-            <near>0.05</near>
-            <far>1.0</far>
-          </clip>
-          <noise>
-            <type>gaussian</type>
-            <mean>0.0</mean>
-            <stddev>0.0</stddev>
-          </noise>
+            <horizontal_fov>1.592</horizontal_fov>
+            <image>
+                <width>1280</width>
+                <height>800</height>
+                <format>R8G8B8</format>
+            </image>
+            <depth_camera>
+            </depth_camera>
+            <clip>
+                <near>0.1</near>
+                <far>100</far>
+            </clip>
         </camera>
-        <plugin name="${name}_frame_controller" filename="libgazebo_ros_openni_kinect.so">
-          <updateRate>25.0</updateRate>
-          <cameraName>${ros_topic}</cameraName>
-          <imageTopicName>rgb/image_raw</imageTopicName>
-          <depthImageTopicName>depth/image_raw</depthImageTopicName>
-          <pointCloudTopicName>depth/points</pointCloudTopicName>
-          <cameraInfoTopicName>rgb/camera_info</cameraInfoTopicName>
-          <depthImageCameraInfoTopicName>depth/camera_info</depthImageCameraInfoTopicName>
-          <frameName>${name}_optical_frame</frameName>
-          <pointCloudCutoff>0.05</pointCloudCutoff>
-          <pointCloudCutoffMax>5.0</pointCloudCutoffMax>
-          <distortionK1>0.0</distortionK1>
-          <distortionK2>0.0</distortionK2>
-          <distortionK3>0.0</distortionK3>
-          <distortionT1>0.0</distortionT1>
-          <distortionT2>0.0</distortionT2>
-          <CxPrime>0.0</CxPrime>
-          <Cx>0.0</Cx>
-          <Cy>0.0</Cy>
-          <focalLength>0.0</focalLength>
-        </plugin>
-      </sensor>
-      <material>IPA/LightGrey</material>
-    </gazebo>
+             <plugin name="camera_controller" filename="libgazebo_ros_openni_kinect.so">
+             <alwaysOn>true</alwaysOn>
+                <updateRate>10.0</updateRate>
+                <cameraName>camera</cameraName>
+                <frameName>camera_depth_optical_frame</frameName>
+            <imageTopicName>color/image_raw</imageTopicName>
+            <depthImageTopicName>depth/color/image_raw</depthImageTopicName>
+            <pointCloudTopicName>depth/color/points</pointCloudTopicName>
+            <cameraInfoTopicName>color/camera_info</cameraInfoTopicName>
+            <depthImageCameraInfoTopicName>depth/camera_info</depthImageCameraInfoTopicName>
+            <pointCloudCutoff>0.4</pointCloudCutoff>
+                <hackBaseline>0.07</hackBaseline>
+                <distortionK1>0.0</distortionK1>
+                <distortionK2>0.0</distortionK2>
+                <distortionK3>0.0</distortionK3>
+                <distortionT1>0.0</distortionT1>
+                <distortionT2>0.0</distortionT2>
+            <CxPrime>0.0</CxPrime>
+            <Cx>0.0</Cx>
+            <Cy>0.0</Cy>
+            <focalLength>0.0</focalLength>
+            </plugin>
+    </sensor>
+  </gazebo>
   </xacro:macro>
 </robot>
