Commit message: fitting komodo model

File: komodo2_description/urdf/komodo2.xacro (robot description, xacro)
@@ -30,5 +30,5 @@
       <geometry>
         <mesh
-          filename="package://robotican_komodo/description/meshes/base_link.STL" />
+          filename="package://komodo2_description/mesh/base_link.STL" />
       </geometry>
       <material
@@ -44,5 +44,5 @@
       <geometry>
         <mesh
-          filename="package://robotican_komodo/description/meshes/base_link.STL" />
+          filename="package://komodo2_description/mesh/base_link.STL" />
       </geometry>
     </collision>
@@ -70,5 +70,5 @@
       <geometry>
         <mesh
-          filename="package://robotican_komodo/description/meshes/wheel_link.STL" />
+          filename="package://komodo2_description/mesh/wheel_link.STL" />
       </geometry>
       <material
@@ -83,5 +83,5 @@
         rpy="${M_PI/2} 0 0" />
       <geometry>
-	<!--  <mesh filename="package://robotican_komodo/description/meshes/wheel_link.STL" /> -->
+	<!--  <mesh filename="package://komodo2_description/mesh/wheel_link.STL" /> -->
 	  <cylinder  length="0.05" radius="0.127"/>
       </geometry>
@@ -123,5 +123,5 @@
       <geometry>
         <mesh
-          filename="package://robotican_komodo/description/meshes/wheel_link.STL" />
+          filename="package://komodo2_description/mesh/wheel_link.STL" />
       </geometry>
       <material
@@ -136,5 +136,5 @@
         rpy="${M_PI/2} 0 0" />
       <geometry>
-	<!--  <mesh filename="package://robotican_komodo/description/meshes/wheel_link.STL" /> -->
+	<!--  <mesh filename="package://komodo2_description/mesh/wheel_link.STL" /> -->
 	  <cylinder  length="0.05" radius="0.127"/>
       </geometry>
@@ -176,5 +176,5 @@
       <geometry>
         <mesh
-          filename="package://robotican_komodo/description/meshes/wheel_link.STL" />
+          filename="package://komodo2_description/mesh/wheel_link.STL" />
       </geometry>
       <material
@@ -189,5 +189,5 @@
         rpy="${M_PI/2} 0 0" />
       <geometry>
-	<!--  <mesh filename="package://robotican_komodo/description/meshes/wheel_link.STL" /> -->
+	<!--  <mesh filename="package://komodo2_description/mesh/wheel_link.STL" /> -->
 	  <cylinder  length="0.05" radius="0.127"/>
       </geometry>
@@ -229,5 +229,5 @@
       <geometry>
         <mesh
-          filename="package://robotican_komodo/description/meshes/wheel_link.STL" />
+          filename="package://komodo2_description/mesh/wheel_link.STL" />
       </geometry>
       <material
@@ -242,5 +242,5 @@
         rpy="${M_PI/2} 0 0" />
       <geometry>
-	<!--  <mesh filename="package://robotican_komodo/description/meshes/wheel_link.STL" /> -->
+	<!--  <mesh filename="package://komodo2_description/mesh/wheel_link.STL" /> -->
 	  <cylinder  length="0.05" radius="0.127"/>
       </geometry>
@@ -273,5 +273,5 @@
       <geometry>
         <mesh
-          filename="package://robotican_komodo/description/meshes/laser_link.STL" />
+          filename="package://komodo2_description/mesh/laser_link.STL" />
       </geometry>
       <material

File: komodo2_description/urdf/komodo2_gazebo.xacro (robot description, xacro)
@@ -13,9 +13,4 @@
     <xacro:arg name="softkinetic" default="false"/>
   <xacro:arg name="depth_camera" default="false"/>
-  <xacro:include filename="$(find robotican_manipulator_h)/models/manipulator_h_gazebo_plugins.xacro" />
-  <!-- SR300 -->
-  <xacro:if value="$(arg sr300)">
-    <xacro:include filename="$(find robotican_common)/gazebo/sr300.xacro" />
-  </xacro:if>
     <!-- softkinetic -->
   <xacro:if value="$(arg softkinetic)">

Commit message: adding komodo2_gazebo folder

File: komodo2_description/urdf/komodo2.xacro (robot description, xacro)
@@ -1,4 +1,4 @@
 <?xml version="1.0"?>
-	<robot xmlns:xacro="http://www.ros.org/wiki/xacro" name="komodo_robot" description="Komodo Robot">
+	<robot xmlns:xacro="http://www.ros.org/wiki/xacro" name="komodo2_robot" description="Komodo2 Robot">
 	<xacro:property name="M_PI" value="3.1415926535897931" />
 <link name="base_footprint"/>
@@ -294,7 +294,7 @@
   </joint>
   <link
-    name="front_cam_link" />
-  <joint
-    name="front_cam_joint"
+    name="rgb_camera_link" />
+  <joint
+    name="rgb_camera_joint"
     type="fixed">
     <origin
@@ -304,5 +304,5 @@
       link="base_link" />
     <child
-      link="front_cam_link" />
+      link="rgb_camera_link" />
     <axis
       xyz="0 0 0" />
@@ -311,5 +311,5 @@
     name="depth_camera_link" />
   <joint
-    name="depth_cam_joint"
+    name="depth_camera_joint"
     type="fixed">
     <origin

File: komodo2_description/urdf/komodo2_gazebo.xacro (robot description, xacro)
@@ -1,24 +1,12 @@
 <?xml version="1.0"?>
-<robot xmlns:xacro="http://www.ros.org/wiki/xacro" name="Komodo" description="Komodo robot">
+<robot xmlns:xacro="http://www.ros.org/wiki/xacro" name="Komodo2" description="Komodo2 robot">
   <xacro:include filename="$(find robotican_komodo)/description/models/komodo.xacro" />
-  <xacro:include filename="$(find robotican_common)/gazebo/softkinetic_camera_ds325.xacro" />
   <xacro:property name="URF_FOV" value="${10.0*M_PI/180}" />
   <xacro:arg name="controllers" default="true"/>
-  <xacro:arg name="front_camera" default="false"/>
+  <xacro:arg name="rgb_camera" default="false"/>
   <xacro:arg name="urf" default="false"/>
   <xacro:arg name="imu" default="false"/>
   <xacro:arg name="gps" default="false"/>
   <xacro:arg name="lidar" default="false"/>
-  <xacro:arg name="sr300" default="false"/>
-    <xacro:arg name="softkinetic" default="false"/>
-  <xacro:arg name="depth_camera" default="false"/>
-    <!-- softkinetic -->
-  <xacro:if value="$(arg softkinetic)">
-     <xacro:softkinetic_gazebo name="softkinetic_camera_rgb" ros_topic="softkinetic_camera"/>
-  </xacro:if>
-  <!-- TODO: Asus -->
-  <xacro:if value="$(arg depth_camera)">
-    <xacro:include filename="$(find robotican_common)/gazebo/asus_xtion_pro_live.xacro" />
-  </xacro:if>
   <!-- Sonars -->
   <xacro:if value="$(arg urf)">
@@ -48,8 +36,8 @@
     <!-- cameras  -->
     <xacro:include filename="$(find robotican_common)/gazebo/camera.xacro" />
-    <xacro:if value="$(arg front_camera)">
-      <xacro:Camera name="front_camera" link="front_cam_link" image_width="640" image_height="480"
+    <xacro:if value="$(arg rgb_camera)">
+    <xacro:Camera name="rgb_camera" link="rgb_camera_link" image_width="640" image_height="480"
         image_format="R8G8B8" clip_near="0.02" clip_far="300" />
-      </xacro:if>
+    </xacro:if>
       <!-- controller manager and hardware interfaces -->
       <xacro:if value="$(arg controllers)">
@@ -60,42 +48,42 @@
         </gazebo>
         <!-- joints -->
-        <transmission name="FL_wheel_joint_trans">
+        <transmission name="front_left_wheel_joint_trans">
           <type>transmission_interface/SimpleTransmission</type>
-          <joint name="FL_wheel_joint">
+          <joint name="front_left_wheel_joint">
             <hardwareInterface>VelocityJointInterface</hardwareInterface>
           </joint>
-          <actuator name="FL_wheel_joint_motor">
+          <actuator name="front_left_wheel_joint_motor">
             <mechanicalReduction>1</mechanicalReduction>
           </actuator>
         </transmission>
-        <transmission name="FR_wheel_joint_trans">
+        <transmission name="front_right_wheel_joint_trans">
           <type>transmission_interface/SimpleTransmission</type>
-          <joint name="FR_wheel_joint">
+          <joint name="front_right_wheel_joint">
             <hardwareInterface>VelocityJointInterface</hardwareInterface>
           </joint>
-          <actuator name="FR_wheel_joint_motor">
+          <actuator name="front_right_wheel_joint_motor">
             <mechanicalReduction>1</mechanicalReduction>
           </actuator>
         </transmission>
-        <transmission name="RL_wheel_joint_trans">
+        <transmission name="rear_left_wheel_joint_trans">
           <type>transmission_interface/SimpleTransmission</type>
-          <joint name="RL_wheel_joint">
+          <joint name="rear_left_wheel_joint">
             <hardwareInterface>VelocityJointInterface</hardwareInterface>
           </joint>
-          <actuator name="RL_wheel_joint_motor">
+          <actuator name="rear_left_wheel_joint_motor">
             <mechanicalReduction>1</mechanicalReduction>
           </actuator>
         </transmission>
-        <transmission name="RR_wheel_joint_trans">
+        <transmission name="rear_right_wheel_joint_trans">
           <type>transmission_interface/SimpleTransmission</type>
-          <joint name="RR_wheel_joint">
+          <joint name="rear_right_wheel_joint">
             <hardwareInterface>VelocityJointInterface</hardwareInterface>
           </joint>
-          <actuator name="RR_wheel_joint_motor">
+          <actuator name="rear_right_wheel_joint_motor">
             <mechanicalReduction>1</mechanicalReduction>
           </actuator>
         </transmission>
       </xacro:if>
-      <gazebo reference="FL_wheel_link">
+      <gazebo reference="front_left_wheel_link">
         <!-- kp and kd for rubber -->
         <kp>1000000.0</kp>
@@ -108,5 +96,5 @@
         <material>Gazebo/Black</material>
       </gazebo>
-      <gazebo reference="FR_wheel_link">
+      <gazebo reference="front_right_wheel_link">
         <!-- kp and kd for rubber -->
         <kp>1000000.0</kp>
@@ -119,5 +107,5 @@
         <material>Gazebo/Black</material>
       </gazebo>
-      <gazebo reference="RL_wheel_link">
+      <gazebo reference="rear_left_wheel_link">
         <!-- kp and kd for rubber -->
         <kp>1000000.0</kp>
@@ -130,5 +118,5 @@
         <material>Gazebo/Black</material>
       </gazebo>
-      <gazebo reference="RR_wheel_link">
+      <gazebo reference="rear_right_wheel_link">
         <!-- kp and kd for rubber -->
         <kp>1000000.0</kp>
@@ -144,20 +132,11 @@
         <material>Gazebo/Grey</material>
       </gazebo>
-      <gazebo reference="FR_urf_link">
+      <gazebo reference="right_urf_link">
         <material>Gazebo/Black</material>
       </gazebo>
-      <gazebo reference="FL_urf_link">
+      <gazebo reference="left_urf_link">
         <material>Gazebo/Black</material>
       </gazebo>
-      <gazebo reference="RR_urf_link">
-        <material>Gazebo/Black</material>
-      </gazebo>
-      <gazebo reference="RL_urf_link">
-        <material>Gazebo/Black</material>
-      </gazebo>
-      <gazebo reference="rear_urf_link">
-        <material>Gazebo/Black</material>
-      </gazebo>
-      <gazebo reference="sr300_link">
+      <gazebo reference="front_urf_link">
         <material>Gazebo/Black</material>
       </gazebo>

Commit message: fitting komodo2_gazebo.xacro

File: komodo2_description/urdf/komodo2.xacro (robot description, xacro)
@@ -294,5 +294,5 @@
   </joint>
   <link
-    name="rgb_camera_link" />
+    name="front_camera_link" />
   <joint
     name="rgb_camera_joint"
@@ -304,5 +304,5 @@
       link="base_link" />
     <child
-      link="rgb_camera_link" />
+      link="camera_link" />
     <axis
       xyz="0 0 0" />

File: komodo2_description/urdf/komodo2_gazebo.xacro (robot description, xacro)
@@ -1,89 +1,83 @@
 <?xml version="1.0"?>
 <robot xmlns:xacro="http://www.ros.org/wiki/xacro" name="Komodo2" description="Komodo2 robot">
-  <xacro:include filename="$(find robotican_komodo)/description/models/komodo.xacro" />
-  <xacro:property name="URF_FOV" value="${10.0*M_PI/180}" />
-  <xacro:arg name="controllers" default="true"/>
-  <xacro:arg name="rgb_camera" default="false"/>
-  <xacro:arg name="urf" default="false"/>
-  <xacro:arg name="imu" default="false"/>
-  <xacro:arg name="gps" default="false"/>
-  <xacro:arg name="lidar" default="false"/>
-  <!-- Sonars -->
-  <xacro:if value="$(arg urf)">
+    <xacro:include filename="$(find robotican_komodo)/description/models/komodo.xacro" />
+    <xacro:property name="URF_FOV" value="${10.0*M_PI/180}" />
+    <xacro:arg name="rgb_camera" default="false"/>
+    <xacro:arg name="depth_camera" default="false"/>
+    <xacro:arg name="lidar" default="false"/>
+    <!-- sonars -->
     <xacro:include filename="$(find komodo2_gazebo)/macros/urf.xacro" />
     <xacro:urf name="left" link="left_urf_link" topic="URF/left" />
     <xacro:urf name="right" link="right_urf_link" topic="URF/right" />
     <xacro:urf name="rear" link="rear_urf_link" topic="URF/rear" />
-  </xacro:if>
-  <!-- hokuyo URG-30LX   -->
-  <xacro:if value="$(arg lidar)">
-    <xacro:include filename="$(find komodo2_gazebo)/macros/hokuyo.xacro" />
-    <xacro:lidar link="laser_link" topic="scan" samples="720" resolution="1" min_angle="-1.5707" max_angle="1.5707" range_min="0.1" range_max="30.0" range_resolution="0.01" />
-  </xacro:if>
-  <!-- GPS   -->
-  <xacro:if value="$(arg gps)">
+    <!-- hokuyo -->
+    <xacro:if value="$(arg lidar)">
+        <xacro:include filename="$(find komodo2_gazebo)/macros/hokuyo.xacro" />
+        <xacro:lidar link="laser_link" topic="scan" samples="720" resolution="1" min_angle="-1.5707" max_angle="1.5707" range_min="0.1" range_max="30.0" range_resolution="0.01" />
+    </xacro:if>
+    <!-- rgb camera  -->
+    <xacro:if value="$(arg rgb_camera)">
+        <xacro:include filename="$(find komodo2_gazebo)/macros/camera.xacro" />
+        <xacro:Camera name="rgb_camera" link="rgb_camera_link" image_width="640" image_height="480" image_format="R8G8B8" clip_near="0.02" clip_far="300" />
+    </xacro:if>
+    <!-- depth camera  -->
+    <xacro:if value="$(arg depth_camera)">
+        <xacro:include filename="$(find komodo2_gazebo)/macros/softkinetic_camera_ds325.xacro" />
+        <xacro:Camera name="depth_camera" link="depth_camera_link" image_width="640" image_height="480" image_format="R8G8B8" clip_near="0.02" clip_far="300" />
+    </xacro:if>
+    <!-- GPS   -->
     <xacro:include filename="$(find komodo2_gazebo)/macros/gps.xacro" />
     <xacro:gps />
-  </xacro:if>
-  <!-- IMU   -->
-  <xacro:if value="$(arg imu)">
+    <!-- IMU   -->
     <xacro:include filename="$(find komodo2_gazebo)/macros/imu.xacro" />
     <xacro:imu link="base_link" imu_offset_x="0" imu_offset_y="0" imu_offset_z="${M_PI}"
-      imu_offset_roll="0" imu_offset_pitch="0"
-      imu_offset_yaw="0" mag_offset_x="0"
-      mag_offset_y="0" mag_offset_z="0" />
-    </xacro:if>
-    <!-- cameras  -->
-    <xacro:include filename="$(find komodo2_gazebo)/macros/camera.xacro" />
-    <xacro:if value="$(arg rgb_camera)">
-    <xacro:Camera name="rgb_camera" link="rgb_camera_link" image_width="640" image_height="480"
-        image_format="R8G8B8" clip_near="0.02" clip_far="300" />
-    </xacro:if>
-      <!-- controller manager and hardware interfaces -->
-      <xacro:if value="$(arg controllers)">
-        <gazebo>
-          <plugin name="gazebo_ros_control" filename="libgazebo_ros_control.so">
-            <robotSimType>gazebo_ros_control/RoboticanRobotHWSim</robotSimType>
-          </plugin>
-        </gazebo>
-        <!-- joints -->
-        <transmission name="front_left_wheel_joint_trans">
-          <type>transmission_interface/SimpleTransmission</type>
-          <joint name="front_left_wheel_joint">
+               imu_offset_roll="0" imu_offset_pitch="0"
+               imu_offset_yaw="0" mag_offset_x="0"
+               mag_offset_y="0" mag_offset_z="0" />
+    <!-- controller manager and hardware interfaces -->
+    <gazebo>
+        <plugin name="gazebo_ros_control" filename="libgazebo_ros_control.so">
+            <robotSimType>gazebo_ros_control/Komodo2HWSim</robotSimType>
+        </plugin>
+    </gazebo>
+    <!-- transmissions -->
+    <transmission name="front_left_wheel_joint_trans">
+        <type>transmission_interface/SimpleTransmission</type>
+        <joint name="front_left_wheel_joint">
             <hardwareInterface>VelocityJointInterface</hardwareInterface>
-          </joint>
-          <actuator name="front_left_wheel_joint_motor">
+        </joint>
+        <actuator name="front_left_wheel_joint_motor">
             <mechanicalReduction>1</mechanicalReduction>
-          </actuator>
-        </transmission>
-        <transmission name="front_right_wheel_joint_trans">
-          <type>transmission_interface/SimpleTransmission</type>
-          <joint name="front_right_wheel_joint">
+        </actuator>
+    </transmission>
+    <transmission name="front_right_wheel_joint_trans">
+        <type>transmission_interface/SimpleTransmission</type>
+        <joint name="front_right_wheel_joint">
             <hardwareInterface>VelocityJointInterface</hardwareInterface>
-          </joint>
-          <actuator name="front_right_wheel_joint_motor">
+        </joint>
+        <actuator name="front_right_wheel_joint_motor">
             <mechanicalReduction>1</mechanicalReduction>
-          </actuator>
-        </transmission>
-        <transmission name="rear_left_wheel_joint_trans">
-          <type>transmission_interface/SimpleTransmission</type>
-          <joint name="rear_left_wheel_joint">
+        </actuator>
+    </transmission>
+    <transmission name="rear_left_wheel_joint_trans">
+        <type>transmission_interface/SimpleTransmission</type>
+        <joint name="rear_left_wheel_joint">
             <hardwareInterface>VelocityJointInterface</hardwareInterface>
-          </joint>
-          <actuator name="rear_left_wheel_joint_motor">
+        </joint>
+        <actuator name="rear_left_wheel_joint_motor">
             <mechanicalReduction>1</mechanicalReduction>
-          </actuator>
-        </transmission>
-        <transmission name="rear_right_wheel_joint_trans">
-          <type>transmission_interface/SimpleTransmission</type>
-          <joint name="rear_right_wheel_joint">
+        </actuator>
+    </transmission>
+    <transmission name="rear_right_wheel_joint_trans">
+        <type>transmission_interface/SimpleTransmission</type>
+        <joint name="rear_right_wheel_joint">
             <hardwareInterface>VelocityJointInterface</hardwareInterface>
-          </joint>
-          <actuator name="rear_right_wheel_joint_motor">
+        </joint>
+        <actuator name="rear_right_wheel_joint_motor">
             <mechanicalReduction>1</mechanicalReduction>
-          </actuator>
-        </transmission>
-      </xacro:if>
-      <gazebo reference="front_left_wheel_link">
+        </actuator>
+    </transmission>
+    <!-- physics -->
+    <gazebo reference="front_left_wheel_link">
         <!-- kp and kd for rubber -->
         <kp>1000000.0</kp>
@@ -95,6 +89,6 @@
         <minDepth>0.00</minDepth>
         <material>Gazebo/Black</material>
-      </gazebo>
-      <gazebo reference="front_right_wheel_link">
+    </gazebo>
+    <gazebo reference="front_right_wheel_link">
         <!-- kp and kd for rubber -->
         <kp>1000000.0</kp>
@@ -106,6 +100,6 @@
         <minDepth>0.00</minDepth>
         <material>Gazebo/Black</material>
-      </gazebo>
-      <gazebo reference="rear_left_wheel_link">
+    </gazebo>
+    <gazebo reference="rear_left_wheel_link">
         <!-- kp and kd for rubber -->
         <kp>1000000.0</kp>
@@ -117,6 +111,6 @@
         <minDepth>0.00</minDepth>
         <material>Gazebo/Black</material>
-      </gazebo>
-      <gazebo reference="rear_right_wheel_link">
+    </gazebo>
+    <gazebo reference="rear_right_wheel_link">
         <!-- kp and kd for rubber -->
         <kp>1000000.0</kp>
@@ -128,16 +122,17 @@
         <minDepth>0.00</minDepth>
         <material>Gazebo/Black</material>
-      </gazebo>
-      <gazebo reference="base_link">
+    </gazebo>
+    <!-- colors -->
+    <gazebo reference="base_link">
         <material>Gazebo/Grey</material>
-      </gazebo>
-      <gazebo reference="right_urf_link">
+    </gazebo>
+    <gazebo reference="right_urf_link">
         <material>Gazebo/Black</material>
-      </gazebo>
-      <gazebo reference="left_urf_link">
+    </gazebo>
+    <gazebo reference="left_urf_link">
         <material>Gazebo/Black</material>
-      </gazebo>
-      <gazebo reference="front_urf_link">
+    </gazebo>
+    <gazebo reference="front_urf_link">
         <material>Gazebo/Black</material>
-      </gazebo>
+    </gazebo>
 </robot>
