Commit message: komodo sim

File: komodo2_description/urdf/komodo2.xacro (robot description, xacro)
@@ -1,20 +1,26 @@
 <?xml version="1.0"?>
-<robot
-  name="komodo2">
+<robot xmlns:xacro="http://www.ros.org/wiki/xacro" name="komodo2_robot" description="Komodo2 Robot">
+	<xacro:property name="M_PI" value="3.1415926535897931" />
+      <link name="base_footprint"/>
+ <joint name="base_footprint_joint" type="fixed">
+    <parent link="base_footprint"/>
+    <child link="base_link"/>
+    <origin xyz="0.00 0.00 0.1275" rpy="0.0 0.0 0.0"/>
+  </joint>
   <link
     name="base_link">
     <inertial>
       <origin
-        xyz="0.0265371254582772 0.000242403640172173 0.0501704404394482"
+        xyz="0.0030152 0.00057861 0.0749"
         rpy="0 0 0" />
       <mass
-        value="1.70660108565618" />
+        value="20.0058" />
       <inertia
-        ixx="0.0285642304866605"
-        ixy="-0.000201185394992359"
-        ixz="-0.000317415309478303"
-        iyy="0.0639136623858303"
-        iyz="-1.60880321018346E-06"
-        izz="0.07625494098217" />
+        ixx="0.025582"
+        ixy="0.0010034"
+        ixz="-0.0041152"
+        iyy="0.086418"
+        iyz="-3.8058E-05"
+        izz="0.091994" />
     </inertial>
     <visual>
@@ -24,10 +30,10 @@
       <geometry>
         <mesh
-          filename="package://komodo2/meshes/base.STL" />
+          filename="package://komodo2_description/mesh/base.STL" />
       </geometry>
       <material
         name="">
         <color
-          rgba="0.792156862745098 0.819607843137255 0.933333333333333 1" />
+          rgba="0.79216 0.81961 0.93333 1" />
       </material>
     </visual>
@@ -38,128 +44,23 @@
       <geometry>
         <mesh
-          filename="package://komodo2/meshes/base.STL" />
+          filename="package://komodo2_description/mesh/base.STL" />
       </geometry>
     </collision>
   </link>
   <link
-    name="footprint_link" />
-  <joint
-    name="footprint_joint"
-    type="fixed">
-    <origin
-      xyz="0 -0.00349999999999995 -0.126"
-      rpy="0 0 0" />
-    <parent
-      link="base_link" />
-    <child
-      link="footprint_link" />
-    <axis
-      xyz="0 0 0" />
-  </joint>
-  <link
-    name="laser_link" />
-  <joint
-    name="laser_joint"
-    type="fixed">
-    <origin
-      xyz="0.233497501055752 0 0.141334654748157"
-      rpy="0 0 0" />
-    <parent
-      link="base_link" />
-    <child
-      link="laser_link" />
-    <axis
-      xyz="0 0 0" />
-  </joint>
-  <link
-    name="front_cam_link" />
-  <joint
-    name="front_cam_joint"
-    type="fixed">
-    <origin
-      xyz="0.257250027816762 0.0875000000000053 0.1"
-      rpy="0 0 0" />
-    <parent
-      link="base_link" />
-    <child
-      link="front_cam_link" />
-    <axis
-      xyz="0 0 0" />
-  </joint>
-  <link
-    name="depth_cam_link" />
-  <joint
-    name="depth_cam_joint"
-    type="fixed">
-    <origin
-      xyz="0.262250027816762 0.00102830288238904 0.0635000000000002"
-      rpy="0 0 0" />
-    <parent
-      link="base_link" />
-    <child
-      link="depth_cam_link" />
-    <axis
-      xyz="0 0 0" />
-  </joint>
-  <link
-    name="right_urf_link" />
-  <joint
-    name="right_urf_joint"
-    type="fixed">
-    <origin
-      xyz="-0.0225419326154781 -0.137249999999995 0.138101776066688"
-      rpy="0 0 0" />
-    <parent
-      link="base_link" />
-    <child
-      link="right_urf_link" />
-    <axis
-      xyz="0 0 0" />
-  </joint>
-  <link
-    name="rear_urf_link" />
-  <joint
-    name="rear_urf_joint"
-    type="fixed">
-    <origin
-      xyz="-0.267499972183238 0.00022860000000516 0.1175936"
-      rpy="0 0 3.14159265358979" />
-    <parent
-      link="base_link" />
-    <child
-      link="rear_urf_link" />
-    <axis
-      xyz="0 0 0" />
-  </joint>
-  <link
-    name="left_urf_link" />
-  <joint
-    name="left_urf_joint"
-    type="fixed">
-    <origin
-      xyz="-0.0220847326154781 0.137250000000005 0.138101776066688"
-      rpy="0 0 0" />
-    <parent
-      link="base_link" />
-    <child
-      link="left_urf_link" />
-    <axis
-      xyz="0 0 0" />
-  </joint>
-  <link
-    name="front_left_wheel_link">
+    name="rear_left_wheel_link">
     <inertial>
       <origin
-        xyz="1.06542009199739E-05 0.00115773372814759 -1.501840532905E-05"
+        xyz="9.8684E-07 -9.3003E-05 -1.8753E-05"
         rpy="0 0 0" />
       <mass
-        value="2.68204072018496" />
+        value="2.6829" />
       <inertia
-        ixx="0.0127575754327221"
-        ixy="1.06323698473979E-06"
-        ixz="1.32400044989008E-06"
-        iyy="0.0232771977739384"
-        iyz="-1.70158762992046E-06"
-        izz="0.0127565430134399" />
+        ixx="0.012758"
+        ixy="8.7952E-09"
+        ixz="-1.0406E-07"
+        iyy="0.023277"
+        iyz="2.0115E-06"
+        izz="0.012755" />
     </inertial>
     <visual>
@@ -169,10 +70,10 @@
       <geometry>
         <mesh
-          filename="package://komodo2/meshes/wheel.STL" />
+          filename="package://komodo2_description/mesh/wheel.STL" />
       </geometry>
       <material
         name="">
         <color
-          rgba="0.792156862745098 0.819607843137255 0.933333333333333 1" />
+          rgba="0.79216 0.81961 0.93333 1" />
       </material>
     </visual>
@@ -180,39 +81,39 @@
       <origin
         xyz="0 0 0"
-        rpy="0 0 0" />
-      <geometry>
-        <mesh
-          filename="package://komodo2/meshes/wheel.STL" />
+        rpy="${M_PI/2} 0 0" />
+      <geometry>
+	<!--  <mesh filename="package://komodo2_description/mesh/wheel.STL" /> -->
+	  <cylinder  length="0.05" radius="0.127"/>
       </geometry>
     </collision>
   </link>
   <joint
-    name="front_left_wheel_joint"
+    name="rear_left_wheel_joint"
     type="continuous">
     <origin
-      xyz="0.173999999999995 0.1869 0"
-      rpy="0 0 0" />
-    <parent
-      link="base_link" />
-    <child
-      link="front_left_wheel_link" />
+      xyz="-0.165 0.18955 0"
+      rpy="0 0 0" />
+    <parent
+      link="base_link" />
+    <child
+      link="rear_left_wheel_link" />
     <axis
       xyz="0 1 0" />
   </joint>
   <link
-    name="rear_left_wheel_link">
+    name="front_left_wheel_link">
     <inertial>
       <origin
-        xyz="0.33001065420092 0.00115773372814756 -1.50184053290035E-05"
+        xyz="9.8687E-07 -9.3003E-05 -1.8753E-05"
         rpy="0 0 0" />
       <mass
-        value="2.68204072018496" />
+        value="2.6829" />
       <inertia
-        ixx="0.0127575754327221"
-        ixy="1.06323698473982E-06"
-        ixz="1.32400044989004E-06"
-        iyy="0.0232771977739384"
-        iyz="-1.70158762992044E-06"
-        izz="0.0127565430134399" />
+        ixx="0.012758"
+        ixy="8.7932E-09"
+        ixz="-1.0406E-07"
+        iyy="0.023277"
+        iyz="2.0115E-06"
+        izz="0.012755" />
     </inertial>
     <visual>
@@ -222,10 +123,10 @@
       <geometry>
         <mesh
-          filename="package://komodo2/meshes/wheel.STL" />
+          filename="package://komodo2_description/mesh/wheel.STL" />
       </geometry>
       <material
         name="">
         <color
-          rgba="0.792156862745098 0.819607843137255 0.933333333333333 1" />
+          rgba="0.79216 0.81961 0.93333 1" />
       </material>
     </visual>
@@ -233,39 +134,39 @@
       <origin
         xyz="0 0 0"
-        rpy="0 0 0" />
-      <geometry>
-        <mesh
-          filename="package://komodo2/meshes/wheel.STL" />
+        rpy="${M_PI/2} 0 0" />
+      <geometry>
+	<!--  <mesh filename="package://komodo2_description/mesh/wheel.STL" /> -->
+	  <cylinder  length="0.05" radius="0.127"/>
       </geometry>
     </collision>
   </link>
   <joint
-    name="rear_left_wheel_joint"
+    name="front_left_wheel_joint"
     type="continuous">
     <origin
-      xyz="-0.156000000000005 0.1869 0"
-      rpy="0 0 0" />
-    <parent
-      link="base_link" />
-    <child
-      link="rear_left_wheel_link" />
+      xyz="0.165 0.18955 0"
+      rpy="0 0 0" />
+    <parent
+      link="base_link" />
+    <child
+      link="front_left_wheel_link" />
     <axis
       xyz="0 1 0" />
   </joint>
   <link
-    name="front_right_wheel_link">
+    name="rear_right_wheel_link">
     <inertial>
       <origin
-        xyz="1.06542009198907E-05 0.374957733728148 -1.50184053290484E-05"
+        xyz="-9.8675E-07 9.3004E-05 -1.8753E-05"
         rpy="0 0 0" />
       <mass
-        value="2.68204072018496" />
+        value="2.6829" />
       <inertia
-        ixx="0.0127575754327221"
-        ixy="1.0632369847399E-06"
-        ixz="1.3240004498902E-06"
-        iyy="0.0232771977739384"
-        iyz="-1.70158762992054E-06"
-        izz="0.0127565430134399" />
+        ixx="0.012758"
+        ixy="8.801E-09"
+        ixz="1.0405E-07"
+        iyy="0.023277"
+        iyz="-2.0115E-06"
+        izz="0.012755" />
     </inertial>
     <visual>
@@ -275,10 +176,10 @@
       <geometry>
         <mesh
-          filename="package://komodo2/meshes/wheel.STL" />
+          filename="package://komodo2_description/mesh/wheel.STL" />
       </geometry>
       <material
         name="">
         <color
-          rgba="0.792156862745098 0.819607843137255 0.933333333333333 1" />
+          rgba="0.79216 0.81961 0.93333 1" />
       </material>
     </visual>
@@ -286,39 +187,39 @@
       <origin
         xyz="0 0 0"
-        rpy="0 0 0" />
-      <geometry>
-        <mesh
-          filename="package://komodo2/meshes/wheel.STL" />
+        rpy="${M_PI/2} 0 0" />
+      <geometry>
+	<!--  <mesh filename="package://komodo2_description/mesh/wheel.STL" /> -->
+	  <cylinder  length="0.05" radius="0.127"/>
       </geometry>
     </collision>
   </link>
   <joint
-    name="front_right_wheel_joint"
+    name="rear_right_wheel_joint"
     type="continuous">
     <origin
-      xyz="0.173999999999995 -0.1869 0"
-      rpy="0 0 0" />
-    <parent
-      link="base_link" />
-    <child
-      link="front_right_wheel_link" />
+      xyz="-0.165 -0.18955 0"
+      rpy="0 0 0" />
+    <parent
+      link="base_link" />
+    <child
+      link="rear_right_wheel_link" />
     <axis
       xyz="0 1 0" />
   </joint>
   <link
-    name="rear_right_wheel_link">
+    name="front_right_wheel_link">
     <inertial>
       <origin
-        xyz="0.33001065420092 0.374957733728148 -1.50184053290297E-05"
+        xyz="-9.867E-07 9.3004E-05 -1.8753E-05"
         rpy="0 0 0" />
       <mass
-        value="2.68204072018496" />
+        value="2.6829" />
       <inertia
-        ixx="0.0127575754327221"
-        ixy="1.06323698473987E-06"
-        ixz="1.32400044989002E-06"
-        iyy="0.0232771977739384"
-        iyz="-1.70158762992054E-06"
-        izz="0.0127565430134399" />
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
File: komodo2_description/urdf/komodo2_gazebo.xacro (robot description, xacro)
@@ -1,86 +1,145 @@
 <?xml version="1.0"?>
-<robot xmlns:xacro="http://www.ros.org/wiki/xacro" name="komodo2_robot" description="ARMadillo2 Robot">
+<robot xmlns:xacro="http://www.ros.org/wiki/xacro" name="Komodo2" description="Komodo robot">
     <xacro:include filename="$(find komodo2_description)/urdf/komodo2.xacro" />
-    <xacro:arg name="depth_cam" default="true"/>
-    <xacro:arg name="rgb_cam" default="30.0"/>
-    <xacro:arg name="urf" default="true"/>
-    <xacro:arg name="imu" default="true"/>
-    <xacro:arg name="gps" default="true"/>
-    <xacro:arg name="lidar" default="true"/>
-    <xacro:arg name="softkinetic" default="true"/>
+    <xacro:include filename="$(find komodo2_gazebo)/macros/camera.xacro" />
+    <xacro:property name="URF_FOV" value="${10.0*M_PI/180}" />
+    <xacro:arg name="controllers" default="true"/>
+    <xacro:arg name="urf" default="false"/>
+    <xacro:arg name="imu" default="false"/>
+    <xacro:arg name="gps" default="false"/>
+    <xacro:arg name="lidar" default="false"/>
+    <xacro:arg name="rgb_cam" default="false"/>
+    <xacro:arg name="depth_cam" default="false"/>
     <!-- softkinetic -->
-    <xacro:if value="$(arg depth_cam)">
-<!--        <xacro:softkinetic_gazebo name="softkinetic_rgb" ros_topic="softkinetic"/> -->
+    <xacro:if value="$(arg rgb_cam)">
+<!--        <xacro:softkinetic_gazebo name="softkinetic_camera_rgb" ros_topic="softkinetic_camera"/> -->
     </xacro:if>
-    <!-- kinect 2 -->
+    <!-- cameras  -->
     <xacro:if value="$(arg rgb_cam)">
-<!--        <xacro:property name="kinect2_hz" value="$(arg kinect2_hz)"/>
-        <xacro:property name="kinect2_hd" value="$(arg kinect2_hd)"/>
-        <xacro:property name="kinect2_qhd" value="$(arg kinect2_qhd)"/>
-        <xacro:property name="kinect2_sd" value="$(arg kinect2_sd)"/>
-        <xacro:include filename="$(find komodo2_gazebo)/macros/kinect2.xacro" />-->
-    </xacro:if>
-    <!-- Sonars -->
-    <xacro:if value="$(arg urf)">
-        <xacro:include filename="$(find komodo2_gazebo)/macros/urf.xacro" />
-        <xacro:urf name="front" link="front_urf_link" topic="URF/front" fov="${10.0*M_PI/180.0}" min="0.2" max="5.0"/>
-    </xacro:if>
-    <!-- hokuyo  utm-30lx -->
-    <xacro:if value="$(arg lidar)">
-        <xacro:include filename="$(find komodo2_gazebo)/macros/hokuyo.xacro" />
-        <xacro:lidar link="laser_link" topic="scan" samples="720" resolution="1" min_angle="-1.5707963" max_angle="1.5707963" range_min="0.1" range_max="30" range_resolution="0.03" />
-    </xacro:if>
-    <!-- GPS   -->
-    <xacro:if value="$(arg gps)">
-        <xacro:include filename="$(find komodo2_gazebo)/macros/gps.xacro" />
-        <xacro:gps link="base_link" hz="5" topic="GPS" lat="31.262218" long="34.80146100" alt="298"/>
-    </xacro:if>
-    <!-- IMU   -->
-    <xacro:if value="$(arg imu)">
-        <xacro:include filename="$(find komodo2_gazebo)/macros/imu.xacro" />
-        <xacro:imu link="base_link" hz="50" topic="IMU" />
-    </xacro:if>
-    <gazebo>
-        <plugin name="gazebo_ros_control" filename="libgazebo_ros_control.so">
-            <robotSimType>gazebo_ros_control/Komodo2RobotHWSim</robotSimType>
-        </plugin>
-    </gazebo>
-    <transmission name="left_wheel_joint_trans">
-        <type>transmission_interface/SimpleTransmission</type>
-        <joint name="left_wheel_joint">
-            <hardwareInterface>VelocityJointInterface</hardwareInterface>
-        </joint>
-        <actuator name="left_wheel_joint_motor">
-            <mechanicalReduction>1</mechanicalReduction>
-        </actuator>
-    </transmission>
-    <transmission name="right_wheel_joint_trans">
-        <type>transmission_interface/SimpleTransmission</type>
-        <joint name="right_wheel_joint">
-            <hardwareInterface>VelocityJointInterface</hardwareInterface>
-        </joint>
-        <actuator name="right_wheel_joint_motor">
-            <mechanicalReduction>1</mechanicalReduction>
-        </actuator>
-    </transmission>
-    <gazebo reference="left_wheel_link">
-        <mu1>1.0</mu1>
-        <mu2>1.0</mu2>
-        <kp>1000000.0</kp>
-        <kd>100.0</kd>
-        <minDepth>0.001</minDepth>
-        <maxVel>1.0</maxVel>
-    </gazebo>
-    <gazebo reference="right_wheel_link">
-        <mu1>1.0</mu1>
-        <mu2>1.0</mu2>
-        <kp>1000000.0</kp>
-        <kd>100.0</kd>
-        <minDepth>0.001</minDepth>
-        <maxVel>1.0</maxVel>
-    </gazebo>
-    <gazebo reference="base_link">
-        <mu1>0.3</mu1>
-        <mu2>0.3</mu2>
-    </gazebo>
-</robot>
+        <xacro:Camera name="rgb_cam" link="rgb_cam_link" image_width="640" image_height="480"
+                      image_format="R8G8B8" clip_near="0.02" clip_far="300" />
+        </xacro:if>
+        <!-- Sonars -->
+        <xacro:if value="$(arg urf)">
+            <xacro:include filename="$(find komodo2_gazebo)/macros/urf.xacro" />
+            <xacro:urf name="left" link="left_urf_link" topic="URF/left" fov="${10.0*M_PI/180.0}" min="0.2" max="5.0"/>
+            <xacro:urf name="right" link="right_urf_link" topic="URF/right" fov="${10.0*M_PI/180.0}" min="0.2" max="5.0"/>
+            <xacro:urf name="rear" link="rear_urf_link" topic="URF/rear" fov="${10.0*M_PI/180.0}" min="0.2" max="5.0"/>
+        </xacro:if>
+        <!-- hokuyo -->
+        <xacro:if value="$(arg lidar)">
+            <xacro:include filename="$(find komodo2_gazebo)/macros/hokuyo.xacro" />
+            <xacro:lidar link="laser_link" topic="scan" samples="720" resolution="1" min_angle="-1.5707" max_angle="1.5707" range_min="0.1" range_max="30.0" range_resolution="0.01" />
+        </xacro:if>
+        <!-- GPS   -->
+        <xacro:if value="$(arg gps)">
+            <xacro:include filename="$(find komodo2_gazebo)/macros/gps.xacro" />
+            <xacro:gps link="base_link" hz="5" topic="GPS" lat="31.262218" long="34.80146100" alt="298"/>
+        </xacro:if>
+        <!-- IMU   -->
+        <xacro:if value="$(arg imu)">
+            <xacro:include filename="$(find komodo2_gazebo)/macros/imu.xacro" />
+            <xacro:imu link="base_link" hz="50" topic="IMU" />
+        </xacro:if>
+            <!-- controller manager and hardware interfaces -->
+            <xacro:if value="$(arg controllers)">
+                <gazebo>
+                    <plugin name="gazebo_ros_control" filename="libgazebo_ros_control.so">
+                        <robotSimType>gazebo_ros_control/Komodo2RobotHWSim</robotSimType>
+                    </plugin>
+                </gazebo>
+                <!-- joints -->
+                <transmission name="front_left_wheel_joint_trans">
+                    <type>transmission_interface/SimpleTransmission</type>
+                    <joint name="front_left_wheel_joint">
+                        <hardwareInterface>VelocityJointInterface</hardwareInterface>
+                    </joint>
+                    <actuator name="front_left_wheel_joint_motor">
+                        <mechanicalReduction>1</mechanicalReduction>
+                    </actuator>
+                </transmission>
+                <transmission name="front_right_wheel_joint_trans">
+                    <type>transmission_interface/SimpleTransmission</type>
+                    <joint name="front_right_wheel_joint">
+                        <hardwareInterface>VelocityJointInterface</hardwareInterface>
+                    </joint>
+                    <actuator name="front_right_wheel_joint_motor">
+                        <mechanicalReduction>1</mechanicalReduction>
+                    </actuator>
+                </transmission>
+                <transmission name="rear_left_wheel_joint_trans">
+                    <type>transmission_interface/SimpleTransmission</type>
+                    <joint name="rear_left_wheel_joint">
+                        <hardwareInterface>VelocityJointInterface</hardwareInterface>
+                    </joint>
+                    <actuator name="rear_left_wheel_joint_motor">
+                        <mechanicalReduction>1</mechanicalReduction>
+                    </actuator>
+                </transmission>
+                <transmission name="rear_right_wheel_joint_trans">
+                    <type>transmission_interface/SimpleTransmission</type>
+                    <joint name="rear_right_wheel_joint">
+                        <hardwareInterface>VelocityJointInterface</hardwareInterface>
+                    </joint>
+                    <actuator name="rear_right_wheel_joint_motor">
+                        <mechanicalReduction>1</mechanicalReduction>
+                    </actuator>
+                </transmission>
+            </xacro:if>
+            <gazebo reference="front_left_wheel_link">
+                <!-- kp and kd for rubber -->
+                <kp>1000000.0</kp>
+                <kd>100.0</kd>
+                <mu1>1.5</mu1>
+                <mu2>1.5</mu2>
+                <fdir1>1 0 0</fdir1>
+                <maxVel>1.0</maxVel>
+                <minDepth>0.00</minDepth>
+                <material>Gazebo/Black</material>
+            </gazebo>
+            <gazebo reference="front_right_wheel_link">
+                <!-- kp and kd for rubber -->
+                <kp>1000000.0</kp>
+                <kd>100.0</kd>
+                <mu1>1.5</mu1>
+                <mu2>1.5</mu2>
+                <fdir1>1 0 0</fdir1>
+                <maxVel>1.0</maxVel>
+                <minDepth>0.00</minDepth>
+                <material>Gazebo/Black</material>
+            </gazebo>
+            <gazebo reference="rear_left_wheel_link">
+                <!-- kp and kd for rubber -->
+                <kp>1000000.0</kp>
+                <kd>100.0</kd>
+                <mu1>1.5</mu1>
+                <mu2>1.5</mu2>
+                <fdir1>1 0 0</fdir1>
+                <maxVel>1.0</maxVel>
+                <minDepth>0.00</minDepth>
+                <material>Gazebo/Black</material>
+            </gazebo>
+            <gazebo reference="rear_right_wheel_link">
+                <!-- kp and kd for rubber -->
+                <kp>1000000.0</kp>
+                <kd>100.0</kd>
+                <mu1>1.5</mu1>
+                <mu2>1.5</mu2>
+                <fdir1>1 0 0</fdir1>
+                <maxVel>1.0</maxVel>
+                <minDepth>0.00</minDepth>
+                <material>Gazebo/Black</material>
+            </gazebo>
+            <gazebo reference="base_link">
+                <material>Gazebo/Grey</material>
+            </gazebo>
+            <gazebo reference="left_urf_link">
+                <material>Gazebo/Black</material>
+            </gazebo>
+            <gazebo reference="rear_urf_link">
+                <material>Gazebo/Black</material>
+            </gazebo>
+            <gazebo reference="right_urf_link">
+                <material>Gazebo/Black</material>
+            </gazebo>
+        </robot>
