Commit message: adding depth cam urdf

File: komodo2_description/urdf/komodo2.xacro (robot description, xacro)
@@ -291,19 +291,4 @@
   </joint>
   <link
-    name="depth_cam_link" />
-  <joint
-    name="depth_cam_joint"
-    type="fixed">
-    <origin
-      xyz="0.25525 0.0006082 0.063584"
-      rpy="0 0 0" />
-    <parent
-      link="base_link" />
-    <child
-      link="depth_cam_link" />
-    <axis
-      xyz="0 0 0" />
-  </joint>
-  <link
     name="rear_urf_link" />
   <joint
@@ -350,59 +335,108 @@
       xyz="0 0 0" />
   </joint>
-<joint name="depth_cam_rgb_joint" type="fixed">
-      <origin xyz="0 0.0185 0" rpy="0 0 0"/>
-      <parent link="depth_cam_link"/>
-      <child link="depth_cam_rgb_frame" />
-    </joint>
-    <link name="depth_cam_rgb_frame">
+<!--
+License: Apache 2.0. See LICENSE file in root directory.
+Copyright(c) 2017 Intel Corporation. All Rights Reserved
+the following is the URDF model for the Intel RealSense 430 camera, in it's
+aluminum peripherial evaluation case.
+-->
+  <!-- depth camera -->
+  <xacro:property name="r430_cam_depth_to_left_ir_offset" value="-0.025"/>
+  <xacro:property name="r430_cam_depth_to_right_ir_offset" value="0.025"/>
+  <xacro:property name="r430_cam_depth_to_fisheye_offset" value="0.042"/>
+  <!-- The following values model the aluminum peripherial case for the
+    R430 camera, with the camera joint represented by the actual
+    peripherial camera tripod mount -->
+  <xacro:property name="r430_cam_width" value="0.105"/>
+  <xacro:property name="r430_cam_height" value="0.039"/>
+  <xacro:property name="r430_cam_depth" value="0.019"/>
+  <xacro:property name="r430_cam_mount_from_center_offset" value=".0275"/>
+  <!-- The following offset is relative the the physical R430 camera peripherial
+    camera tripod mount -->
+  <xacro:property name="r430_cam_depth_px" value="0.00"/>
+  <xacro:property name="r430_cam_depth_py" value="-0.035"/>
+  <xacro:property name="r430_cam_depth_pz" value="0.028"/>
+             <!-- camera body, with origin at bottom screw mount -->
+    <joint name="camera_joint" type="fixed">
+      <origin
+      xyz="0.25525 0.0006082 0.063584"
+      rpy="0 0 0" />
+    <parent
+      link="base_link" />
+      <child link="camera_link" />
+    </joint>
+    <link name="camera_link">
+      <visual>
+      <origin xyz="0 ${-r430_cam_mount_from_center_offset} ${r430_cam_height/2}" rpy="${M_PI/2} 0 ${M_PI/2}"/>
+        <geometry>
+          <box size="${r430_cam_width} ${r430_cam_height} ${r430_cam_depth}"/>
+          <!--<mesh filename="package://realsense_ros_camera/meshes/r430/r430.dae" />-->
+        </geometry>
+        <material name="aluminum"/>
+      </visual>
+      <collision>
+        <origin xyz="0.0 0.0 ${r430_cam_height/2}" rpy="0 0 0"/>
+        <geometry>
+        <box size="${r430_cam_depth} ${r430_cam_width} ${r430_cam_height}"/>
+        </geometry>
+      </collision>
       <inertial>
-	<mass value="0.001" />
-	<origin xyz="0 0 0" />
-	<inertia ixx="0.0001" ixy="0.0" ixz="0.0"
-	  iyy="0.0001" iyz="0.0"
-	  izz="0.0001" />
-	</inertial>
-      </link>
-      <joint name="depth_cam_rgb_optical_joint" type="fixed">
-	<origin xyz="0 0 0" rpy="${-M_PI/2} 0 ${-M_PI/2}" />
-	<parent link="depth_cam_rgb_frame" />
-	<child link="depth_cam_rgb_optical_frame" />
-      </joint>
-      <link name="depth_cam_rgb_optical_frame">
-	<inertial>
-	  <mass value="0.001" />
-	  <origin xyz="0 0 0" />
-	  <inertia ixx="0.0001" ixy="0.0" ixz="0.0"
-	    iyy="0.0001" iyz="0.0"
-	    izz="0.0001" />
-	  </inertial>
-	</link>
-	<joint name="depth_cam_depth_joint" type="fixed">
-	  <origin xyz="0 0.0445 0" rpy="0 0 0" />
-	  <parent link="depth_cam_link" />
-	  <child link="depth_cam_depth_frame" />
-	</joint>
-	<link name="depth_cam_depth_frame">
-	  <inertial>
-	    <mass value="0.001" />
-	    <origin xyz="0 0 0" />
-	    <inertia ixx="0.0001" ixy="0.0" ixz="0.0"
-	      iyy="0.0001" iyz="0.0"
-	      izz="0.0001" />
-	    </inertial>
-	  </link>
-	  <joint name="depth_cam_depth_optical_joint" type="fixed">
-	    <origin xyz="0 0 0" rpy="${-M_PI/2} 0 ${-M_PI/2}" />
-	    <parent link="depth_cam_depth_frame" />
-	    <child link="depth_cam_depth_optical_frame" />
-	  </joint>
-	  <link name="depth_cam_depth_optical_frame">
-	    <inertial>
-	      <mass value="0.001" />
-	      <origin xyz="0 0 0" />
-	      <inertia ixx="0.0001" ixy="0.0" ixz="0.0"
-		iyy="0.0001" iyz="0.0"
-		izz="0.0001" />
-	      </inertial>
-	    </link>
+        <!-- The following are not reliable values, and should not be used for modeling -->
+        <mass value="0.564" />
+        <origin xyz="0 0 0" />
+        <inertia ixx="0.003881243" ixy="0.0" ixz="0.0" iyy="0.000498940" iyz="0.0" izz="0.003879257" />
+      </inertial>
+    </link>
+    <!-- camera depth joints and links -->
+    <joint name="camera_depth_joint" type="fixed">
+      <origin xyz="${r430_cam_depth_px} ${r430_cam_depth_py} ${r430_cam_depth_pz}" rpy="0 0 0"/>
+      <parent link="camera_link"/>
+      <child link="camera_depth_frame" />
+    </joint>
+    <link name="camera_depth_frame"/>
+    <joint name="camera_depth_optical_joint" type="fixed">
+      <origin xyz="0 0 0" rpy="${-M_PI/2} 0 ${-M_PI/2}" />
+      <parent link="camera_depth_frame" />
+      <child link="camera_depth_optical_frame" />
+    </joint>
+    <link name="camera_depth_optical_frame"/>
+    <!-- camera left IR joints and links -->
+    <joint name="camera_left_ir_joint" type="fixed">
+      <origin xyz="0 ${r430_cam_depth_to_left_ir_offset} 0" rpy="0 0 0" />
+      <parent link="camera_depth_frame" />
+      <child link="camera_left_ir_frame" />
+    </joint>
+    <link name="camera_left_ir_frame"/>
+    <joint name="camera_left_ir_optical_joint" type="fixed">
+      <origin xyz="0 0 0" rpy="${-M_PI/2} 0 ${-M_PI/2}" />
+      <parent link="camera_left_ir_frame" />
+      <child link="camera_left_ir_optical_frame" />
+    </joint>
+    <link name="camera_left_ir_optical_frame"/>
+    <!-- camera right IR joints and links -->
+    <joint name="camera_right_ir_joint" type="fixed">
+      <origin xyz="0 ${r430_cam_depth_to_right_ir_offset} 0" rpy="0 0 0" />
+      <parent link="camera_depth_frame" />
+      <child link="camera_right_ir_frame" />
+    </joint>
+    <link name="camera_right_ir_frame"/>
+    <joint name="camera_right_ir_optical_joint" type="fixed">
+      <origin xyz="0 0 0" rpy="${-M_PI/2} 0 ${-M_PI/2}" />
+      <parent link="camera_right_ir_frame" />
+      <child link="camera_right_ir_optical_frame" />
+    </joint>
+    <link name="camera_right_ir_optical_frame"/>
+    <!-- camera fisheye joints and links -->
+    <joint name="camera_fisheye_joint" type="fixed">
+      <origin xyz="0 ${r430_cam_depth_to_fisheye_offset} 0" rpy="0 0 0" />
+      <parent link="camera_depth_frame" />
+      <child link="camera_fisheye_frame" />
+    </joint>
+    <link name="camera_fisheye_frame"/>
+    <joint name="camera_fisheye_optical_joint" type="fixed">
+      <origin xyz="0 0 0" rpy="${-M_PI/2} 0 ${-M_PI/2}" />
+      <parent link="camera_fisheye_frame" />
+      <child link="camera_fisheye_optical_frame" />
+    </joint>
+    <link name="camera_fisheye_optical_frame"/>
 </robot>

Commit message: fixed flipping robot when driving in gazebo

File: komodo2_description/urdf/komodo2.xacro (robot description, xacro)
@@ -55,13 +55,13 @@
         rpy="0 0 0" />
       <mass
-        value="2.6829" />
+        value="1.8524" />
       <inertia
-        ixx="0.012758"
-        ixy="8.7952E-09"
-        ixz="-1.0406E-07"
-        iyy="0.023277"
-        iyz="2.0115E-06"
-        izz="0.012755" />
-    </inertial>
+        ixx="0.0069046"
+        ixy="-3.8717E-08"
+        ixz="2.0707E-07"
+        iyy="0.17"
+        iyz="-1.0124E-07"
+        izz="0.0069054" />
+      </inertial>
     <visual>
       <origin
@@ -100,4 +100,7 @@
     <axis
       xyz="0 1 0" />
+    <limit
+      effort="0.4"
+      velocity="10.0" />
   </joint>
   <link
@@ -108,13 +111,13 @@
         rpy="0 0 0" />
       <mass
-        value="2.6829" />
+        value="1.8524" />
       <inertia
-        ixx="0.012758"
-        ixy="8.7932E-09"
-        ixz="-1.0406E-07"
-        iyy="0.023277"
-        iyz="2.0115E-06"
-        izz="0.012755" />
-    </inertial>
+        ixx="0.0069046"
+        ixy="-3.8717E-08"
+        ixz="2.0707E-07"
+        iyy="0.17"
+        iyz="-1.0124E-07"
+        izz="0.0069054" />
+      </inertial>
     <visual>
       <origin
@@ -153,4 +156,7 @@
     <axis
       xyz="0 1 0" />
+    <limit
+      effort="0.4"
+      velocity="10.0" />
   </joint>
   <link
@@ -161,12 +167,12 @@
         rpy="0 0 0" />
       <mass
-        value="2.6829" />
+        value="1.8524" />
       <inertia
-        ixx="0.012758"
-        ixy="8.801E-09"
-        ixz="1.0405E-07"
-        iyy="0.023277"
-        iyz="-2.0115E-06"
-        izz="0.012755" />
+        ixx="0.0069046"
+        ixy="-3.8717E-08"
+        ixz="-2.0707E-07"
+        iyy="0.17"
+        iyz="1.0124E-07"
+        izz="0.0069054" />
     </inertial>
     <visual>
@@ -206,4 +212,7 @@
     <axis
       xyz="0 1 0" />
+    <limit
+      effort="0.4"
+      velocity="10.0" />
   </joint>
   <link
@@ -214,12 +223,12 @@
         rpy="0 0 0" />
       <mass
-        value="2.6829" />
+        value="1.8524" />
       <inertia
-        ixx="0.012758"
-        ixy="8.8036E-09"
-        ixz="1.0405E-07"
-        iyy="0.023277"
-        iyz="-2.0115E-06"
-        izz="0.012755" />
+        ixx="0.0069046"
+        ixy="-3.8717E-08"
+        ixz="-2.0707E-07"
+        iyy="0.17"
+        iyz="1.0124E-07"
+        izz="0.0069054" />
     </inertial>
     <visual>
@@ -259,4 +268,7 @@
     <axis
       xyz="0 1 0" />
+    <limit
+      effort="0.4"
+      velocity="10.0" />
   </joint>
   <link
@@ -274,4 +286,7 @@
     <axis
       xyz="0 0 0" />
+    <limit
+      effort="0.4"
+      velocity="10.0" />
   </joint>
   <link

File: komodo2_description/urdf/komodo2_gazebo.xacro (robot description, xacro)
@@ -87,7 +87,14 @@
                 </transmission>
             </xacro:if>
+            <!--<kp>1000000.0</kp>
+                <kd>100.0</kd>
+                <mu1>1.5</mu1>
+                <mu2>1.5</mu2>
+                <fdir1>1 0 0</fdir1>
+                <maxVel>1.0</maxVel>
+                <minDepth>0.00</minDepth> -->
             <gazebo reference="front_left_wheel_link">
                 <!-- kp and kd for rubber -->
-                <kp>1000000.0</kp>
+               <kp>1000000.0</kp>
                 <kd>100.0</kd>
                 <mu1>1.5</mu1>
@@ -99,6 +106,6 @@
             </gazebo>
             <gazebo reference="front_right_wheel_link">
-                <!-- kp and kd for rubber -->
-                <kp>1000000.0</kp>
+              <!-- kp and kd for rubber -->
+              <kp>1000000.0</kp>
                 <kd>100.0</kd>
                 <mu1>1.5</mu1>
@@ -110,6 +117,6 @@
             </gazebo>
             <gazebo reference="rear_left_wheel_link">
-                <!-- kp and kd for rubber -->
-                <kp>1000000.0</kp>
+               <!-- kp and kd for rubber -->
+              <kp>1000000.0</kp>
                 <kd>100.0</kd>
                 <mu1>1.5</mu1>
@@ -121,6 +128,6 @@
             </gazebo>
             <gazebo reference="rear_right_wheel_link">
-                <!-- kp and kd for rubber -->
-                <kp>1000000.0</kp>
+           <!-- kp and kd for rubber -->
+               <kp>1000000.0</kp>
                 <kd>100.0</kd>
                 <mu1>1.5</mu1>

Commit message: fixed depth cam origins in urdf

File: komodo2_description/urdf/komodo2.xacro (robot description, xacro)
@@ -355,55 +355,19 @@
 the following is the URDF model for the Intel RealSense 430 camera, in it's
 aluminum peripherial evaluation case.
+Edited by RoboTiCan
 -->
-  <!-- depth camera -->
-  <xacro:property name="r430_cam_depth_to_left_ir_offset" value="-0.025"/>
-  <xacro:property name="r430_cam_depth_to_right_ir_offset" value="0.025"/>
-  <xacro:property name="r430_cam_depth_to_fisheye_offset" value="0.042"/>
-  <!-- The following values model the aluminum peripherial case for the
-    R430 camera, with the camera joint represented by the actual
-    peripherial camera tripod mount -->
-  <xacro:property name="r430_cam_width" value="0.105"/>
-  <xacro:property name="r430_cam_height" value="0.039"/>
-  <xacro:property name="r430_cam_depth" value="0.019"/>
-  <xacro:property name="r430_cam_mount_from_center_offset" value=".0275"/>
-  <!-- The following offset is relative the the physical R430 camera peripherial
-    camera tripod mount -->
-  <xacro:property name="r430_cam_depth_px" value="0.00"/>
-  <xacro:property name="r430_cam_depth_py" value="-0.035"/>
-  <xacro:property name="r430_cam_depth_pz" value="0.028"/>
-             <!-- camera body, with origin at bottom screw mount -->
+  <link
+    name="camera_link" />
     <joint name="camera_joint" type="fixed">
-      <origin
-      xyz="0.25525 0.0006082 0.063584"
-      rpy="0 0 0" />
-    <parent
-      link="base_link" />
-      <child link="camera_link" />
-    </joint>
-    <link name="camera_link">
-      <visual>
-      <origin xyz="0 ${-r430_cam_mount_from_center_offset} ${r430_cam_height/2}" rpy="${M_PI/2} 0 ${M_PI/2}"/>
-        <geometry>
-          <box size="${r430_cam_width} ${r430_cam_height} ${r430_cam_depth}"/>
-          <!--<mesh filename="package://realsense_ros_camera/meshes/r430/r430.dae" />-->
-        </geometry>
-        <material name="aluminum"/>
-      </visual>
-      <collision>
-        <origin xyz="0.0 0.0 ${r430_cam_height/2}" rpy="0 0 0"/>
-        <geometry>
-        <box size="${r430_cam_depth} ${r430_cam_width} ${r430_cam_height}"/>
-        </geometry>
-      </collision>
-      <inertial>
-        <!-- The following are not reliable values, and should not be used for modeling -->
-        <mass value="0.564" />
-        <origin xyz="0 0 0" />
-        <inertia ixx="0.003881243" ixy="0.0" ixz="0.0" iyy="0.000498940" iyz="0.0" izz="0.003879257" />
-      </inertial>
-    </link>
+        <origin
+        xyz="0.25525 0.0006082 0.063584"
+        rpy="0 0 0" />
+    <parent
+        link="base_link" />
+        <child link="camera_link" />
+    </joint>
     <!-- camera depth joints and links -->
     <joint name="camera_depth_joint" type="fixed">
-      <origin xyz="${r430_cam_depth_px} ${r430_cam_depth_py} ${r430_cam_depth_pz}" rpy="0 0 0"/>
+      <origin xyz="0 -0.0122 0" rpy="0 0 0"/>
       <parent link="camera_link"/>
       <child link="camera_depth_frame" />
@@ -418,6 +382,6 @@
     <!-- camera left IR joints and links -->
     <joint name="camera_left_ir_joint" type="fixed">
-      <origin xyz="0 ${r430_cam_depth_to_left_ir_offset} 0" rpy="0 0 0" />
-      <parent link="camera_depth_frame" />
+      <origin xyz="0 -0.0322 0" rpy="0 0 0" />
+      <parent link="camera_link" />
       <child link="camera_left_ir_frame" />
     </joint>
@@ -431,6 +395,6 @@
     <!-- camera right IR joints and links -->
     <joint name="camera_right_ir_joint" type="fixed">
-      <origin xyz="0 ${r430_cam_depth_to_right_ir_offset} 0" rpy="0 0 0" />
-      <parent link="camera_depth_frame" />
+      <origin xyz="0 0.0178 0" rpy="0 0 0" />
+      <parent link="camera_link" />
       <child link="camera_right_ir_frame" />
     </joint>
@@ -444,6 +408,6 @@
     <!-- camera fisheye joints and links -->
     <joint name="camera_fisheye_joint" type="fixed">
-      <origin xyz="0 ${r430_cam_depth_to_fisheye_offset} 0" rpy="0 0 0" />
-      <parent link="camera_depth_frame" />
+      <origin xyz="0 0.0322 0" rpy="0 0 0" />
+      <parent link="camera_link" />
       <child link="camera_fisheye_frame" />
     </joint>

Commit message: added sick laser and model, added asus xition pro live

File: komodo2_description/urdf/komodo2.xacro (robot description, xacro)
@@ -272,11 +272,25 @@
       velocity="32.0" />
   </joint>
-  <link
-    name="laser_link" />
+  <link name="laser_link" >
+    <visual>
+      <origin
+        xyz="0 0 0"
+        rpy="0 0 0" />
+      <geometry>
+        <mesh
+          filename="package://lms1xx/meshes/sick-lms1xx.stl" />
+      </geometry>
+      <material
+        name="">
+        <color
+          rgba="0.79216 0.81961 0.93333 1" />
+      </material>
+    </visual>
+    </link>
   <joint
     name="laser_joint"
     type="fixed">
     <origin
-      xyz="0.233497501055752 0 0.141334654748157"
+      xyz="0.230497501055752 0 0.318"
       rpy="0 0 0" />
     <parent
@@ -350,11 +364,4 @@
       xyz="0 0 0" />
   </joint>
-<!--
-License: Apache 2.0. See LICENSE file in root directory.
-Copyright(c) 2017 Intel Corporation. All Rights Reserved
-the following is the URDF model for the Intel RealSense 430 camera, in it's
-aluminum peripherial evaluation case.
-Edited by RoboTiCan
--->
   <link
     name="camera_link" />
@@ -367,11 +374,49 @@
         <child link="camera_link" />
     </joint>
-    <!-- camera depth joints and links -->
+      <xacro:property name="asus_xtion_pro_depth_rel_rgb_py" value="0.0480" />
+  <xacro:property name="asus_xtion_pro_cam_rel_rgb_py"   value="0.0220" />
+    <joint name="camera_rgb_joint" type="fixed">
+      <origin xyz="0 ${asus_xtion_pro_cam_rel_rgb_py} 0"
+              rpy="0 0 0"/>
+      <parent link="camera_link"/>
+      <child link="camera_rgb_frame"/>
+    </joint>
+    <link name="camera_rgb_frame">
+      <inertial>
+        <mass value="0.001" />
+        <origin xyz="0 0 0" />
+        <inertia ixx="0.0001" ixy="0.0" ixz="0.0"
+          iyy="0.0001" iyz="0.0"
+          izz="0.0001" />
+      </inertial>
+    </link>
+    <joint name="camera_rgb_optical_joint" type="fixed">
+      <origin xyz="0 0 0" rpy="${-M_PI/2} 0 ${-M_PI/2}" />
+      <parent link="camera_rgb_frame" />
+      <child link="camera_rgb_optical_frame" />
+    </joint>
+    <link name="camera_rgb_optical_frame">
+      <inertial>
+        <mass value="0.001" />
+        <origin xyz="0 0 0" />
+        <inertia ixx="0.0001" ixy="0.0" ixz="0.0"
+          iyy="0.0001" iyz="0.0"
+          izz="0.0001" />
+      </inertial>
+    </link>
     <joint name="camera_depth_joint" type="fixed">
-      <origin xyz="0 -0.0122 0" rpy="0 0 0"/>
-      <parent link="camera_link"/>
+      <origin xyz="0 ${asus_xtion_pro_depth_rel_rgb_py} 0" rpy="0 0 0" />
+      <parent link="camera_link" />
       <child link="camera_depth_frame" />
     </joint>
-    <link name="camera_depth_frame"/>
+    <link name="camera_depth_frame">
+      <inertial>
+        <mass value="0.01" />
+        <origin xyz="0 0 0" />
+        <inertia ixx="0.001" ixy="0.0" ixz="0.0"
+          iyy="0.001" iyz="0.0"
+          izz="0.001" />
+      </inertial>
+    </link>
     <joint name="camera_depth_optical_joint" type="fixed">
       <origin xyz="0 0 0" rpy="${-M_PI/2} 0 ${-M_PI/2}" />
@@ -379,43 +424,12 @@
       <child link="camera_depth_optical_frame" />
     </joint>
-    <link name="camera_depth_optical_frame"/>
-    <!-- camera left IR joints and links -->
-    <joint name="camera_left_ir_joint" type="fixed">
-      <origin xyz="0 -0.0322 0" rpy="0 0 0" />
-      <parent link="camera_link" />
-      <child link="camera_left_ir_frame" />
-    </joint>
-    <link name="camera_left_ir_frame"/>
-    <joint name="camera_left_ir_optical_joint" type="fixed">
-      <origin xyz="0 0 0" rpy="${-M_PI/2} 0 ${-M_PI/2}" />
-      <parent link="camera_left_ir_frame" />
-      <child link="camera_left_ir_optical_frame" />
-    </joint>
-    <link name="camera_left_ir_optical_frame"/>
-    <!-- camera right IR joints and links -->
-    <joint name="camera_right_ir_joint" type="fixed">
-      <origin xyz="0 0.0178 0" rpy="0 0 0" />
-      <parent link="camera_link" />
-      <child link="camera_right_ir_frame" />
-    </joint>
-    <link name="camera_right_ir_frame"/>
-    <joint name="camera_right_ir_optical_joint" type="fixed">
-      <origin xyz="0 0 0" rpy="${-M_PI/2} 0 ${-M_PI/2}" />
-      <parent link="camera_right_ir_frame" />
-      <child link="camera_right_ir_optical_frame" />
-    </joint>
-    <link name="camera_right_ir_optical_frame"/>
-    <!-- camera fisheye joints and links -->
-    <joint name="camera_fisheye_joint" type="fixed">
-      <origin xyz="0 0.0322 0" rpy="0 0 0" />
-      <parent link="camera_link" />
-      <child link="camera_fisheye_frame" />
-    </joint>
-    <link name="camera_fisheye_frame"/>
-    <joint name="camera_fisheye_optical_joint" type="fixed">
-      <origin xyz="0 0 0" rpy="${-M_PI/2} 0 ${-M_PI/2}" />
-      <parent link="camera_fisheye_frame" />
-      <child link="camera_fisheye_optical_frame" />
-    </joint>
-    <link name="camera_fisheye_optical_frame"/>
+    <link name="camera_depth_optical_frame">
+      <inertial>
+        <mass value="0.001" />
+        <origin xyz="0 0 0" />
+        <inertia ixx="0.0001" ixy="0.0" ixz="0.0"
+          iyy="0.0001" iyz="0.0"
+          izz="0.0001" />
+      </inertial>
+</link>
 </robot>

File: komodo2_description/urdf/komodo2_gazebo.xacro (robot description, xacro)
@@ -17,6 +17,5 @@
         </xacro:if>
         <xacro:if value="$(arg depth_cam)">
-           <xacro:include filename="$(find komodo2_gazebo)/macros/depth_cam.xacro" />
-            <xacro:softkinetic_gazebo name="softkinetic_rgb" ros_topic="softkinetic"/>
+           <xacro:include filename="$(find komodo2_gazebo)/macros/asus_xiton_pro_live_depth_cam.xacro" />
         </xacro:if>
         <!-- Sonars -->

Commit message: changed imu

File: komodo2_description/urdf/komodo2.xacro (robot description, xacro)
@@ -272,25 +272,11 @@
       velocity="32.0" />
   </joint>
-  <link name="laser_link" >
-    <visual>
-      <origin
-        xyz="0 0 0"
-        rpy="0 0 0" />
-      <geometry>
-        <mesh
-          filename="package://lms1xx/meshes/sick-lms1xx.stl" />
-      </geometry>
-      <material
-        name="">
-        <color
-          rgba="0.79216 0.81961 0.93333 1" />
-      </material>
-    </visual>
-    </link>
+  <link
+    name="laser_link" />
   <joint
     name="laser_joint"
     type="fixed">
     <origin
-      xyz="0.230497501055752 0 0.318"
+      xyz="0.233497501055752 0 0.141334654748157"
       rpy="0 0 0" />
     <parent
@@ -303,5 +289,5 @@
       effort="0.4"
       velocity="32.0" />
-  </joint>
+</joint>
   <link
     name="rgb_cam_link" />
